Commit message: 完成仿真模型加载与控制器加载,还不能行走

File: src/sim_dog/edu_description/urdf/edu_mujoco.urdf (robot description, URDF)
Before this commit: robot edu_urdf, 20 links, 19 joints
Links:
- link FL_ABAD_LINK: geometry collision mesh filename=package://edu_description/meshes/FL_ABAD_LINK.STL; visual mesh filename=package://edu_description/meshes/FL_ABAD_LINK.STL
- link FL_FOOT_LINK: geometry collision mesh filename=package://edu_description/meshes/FL_FOOT_LINK.STL; visual mesh filename=package://edu_description/meshes/FL_FOOT_LINK.STL
- link FL_HIP_LINK: geometry collision mesh filename=package://edu_description/meshes/FL_HIP_LINK.STL; visual mesh filename=package://edu_description/meshes/FL_HIP_LINK.STL
- link FL_KNEE_LINK: geometry collision mesh filename=package://edu_description/meshes/FL_KNEE_LINK.STL; visual mesh filename=package://edu_description/meshes/FL_KNEE_LINK.STL
- link FR_ABAD_LINK: geometry collision mesh filename=package://edu_description/meshes/FR_ABAD_LINK.STL; visual mesh filename=package://edu_description/meshes/FR_ABAD_LINK.STL
- link FR_FOOT_LINK: geometry collision mesh filename=package://edu_description/meshes/FR_FOOT_LINK.STL; visual mesh filename=package://edu_description/meshes/FR_FOOT_LINK.STL
- link FR_HIP_LINK: geometry collision mesh filename=package://edu_description/meshes/FR_HIP_LINK.STL; visual mesh filename=package://edu_description/meshes/FR_HIP_LINK.STL
- link FR_KNEE_LINK: geometry collision mesh filename=package://edu_description/meshes/FR_KNEE_LINK.STL; visual mesh filename=package://edu_description/meshes/FR_KNEE_LINK.STL
- link RL_ABAD_LINK: geometry collision mesh filename=package://edu_description/meshes/RL_ABAD_LINK.STL; visual mesh filename=package://edu_description/meshes/RL_ABAD_LINK.STL
- link RL_FOOT_LINK: geometry collision mesh filename=package://edu_description/meshes/RL_FOOT_LINK.STL; visual mesh filename=package://edu_description/meshes/RL_FOOT_LINK.STL
- link RL_HIP_LINK: geometry collision mesh filename=package://edu_description/meshes/RL_HIP_LINK.STL; visual mesh filename=package://edu_description/meshes/RL_HIP_LINK.STL
- link RL_KNEE_LINK: geometry collision mesh filename=package://edu_description/meshes/RL_KNEE_LINK.STL; visual mesh filename=package://edu_description/meshes/RL_KNEE_LINK.STL
- link RR_ABAD_LINK: geometry collision mesh filename=package://edu_description/meshes/RR_ABAD_LINK.STL; visual mesh filename=package://edu_description/meshes/RR_ABAD_LINK.STL
- link RR_FOOT_LINK: geometry collision mesh filename=package://edu_description/meshes/RR_FOOT_LINK.STL; visual mesh filename=package://edu_description/meshes/RR_FOOT_LINK.STL
- link RR_HIP_LINK: geometry collision mesh filename=package://edu_description/meshes/RR_HIP_LINK.STL; visual mesh filename=package://edu_description/meshes/RR_HIP_LINK.STL
- link RR_KNEE_LINK: geometry collision mesh filename=package://edu_description/meshes/RR_KNEE_LINK.STL; visual mesh filename=package://edu_description/meshes/RR_KNEE_LINK.STL
- link base_link: geometry collision mesh filename=package://edu_description/meshes/BASE_LINK.STL; visual mesh filename=package://edu_description/meshes/BASE_LINK.STL

Commit message: 修改足底碰撞模型为球形，并调整位置以更好地匹配实际情况。

File: src/sim_dog/edu_description/urdf/edu_mujoco.urdf (robot description, URDF)
Before this commit: robot edu_urdf, 20 links, 19 joints
Links:
- link FL_FOOT_LINK: geometry collision sphere radius=0.022; visual mesh filename=package://edu_description/meshes/FL_FOOT_LINK.STL
- link FR_FOOT_LINK: geometry collision sphere radius=0.022; visual mesh filename=package://edu_description/meshes/FR_FOOT_LINK.STL
- link RL_FOOT_LINK: geometry collision sphere radius=0.022; visual mesh filename=package://edu_description/meshes/RL_FOOT_LINK.STL
- link RR_FOOT_LINK: geometry collision sphere radius=0.022; visual mesh filename=package://edu_description/meshes/RR_FOOT_LINK.STL
